Commit message: Added rerun for keyboard control

File: so101/so101.urdf (robot description, URDF)
Before this commit: robot so101, 8 links, 7 joints
Links:
- removed link base_link
- removed link gripper_frame_link
- removed link gripper_link
- removed link lower_arm_link
- removed link moving_jaw_so101_v1_link
- removed link shoulder_link
- removed link upper_arm_link
- removed link wrist_link
- added link Base, mass 0.147; collision mesh filename=assets/Base.stl; visual mesh filename=assets/Base.stl
- added link Fixed_Jaw, mass 0.0929859; collision mesh filename=assets/Fixed_Jaw_Collision_1.stl; collision mesh filename=assets/Fixed_Jaw_Collision_2.stl
- added link Lower_Arm, mass 0.147968; collision mesh filename=assets/Lower_Arm.stl; visual mesh filename=assets/Lower_Arm.stl
- added link Moving_Jaw, mass 0.0202444; collision mesh filename=assets/Moving_Jaw_Collision_1.stl; collision mesh filename=assets/Moving_Jaw_Collision_2.stl
- added link Rotation_Pitch, mass 0.119226; collision mesh filename=assets/Rotation_Pitch.stl; visual mesh filename=assets/Rotation_Pitch.stl
- added link Upper_Arm, mass 0.162409; collision mesh filename=assets/Upper_Arm.stl; visual mesh filename=assets/Upper_Arm.stl
- added link Wrist_Pitch_Roll, mass 0.0661321; collision mesh filename=assets/Wrist_Pitch_Roll.stl; visual mesh filename=assets/Wrist_Pitch_Roll.stl
Joints:
- removed joint elbow_flex
- removed joint gripper
- removed joint gripper_frame_joint
- removed joint shoulder_lift
- removed joint shoulder_pan
- removed joint wrist_flex
- removed joint wrist_roll
- added joint Elbow: type revolute, parent Upper_Arm, child Lower_Arm, origin xyz=0 0.11257 0.028 rpy=-1.5708 0 0, axis 1 0 0, limit lower=0 upper=3.14159 effort=35 velocity=10
- added joint Jaw: type revolute, parent Fixed_Jaw, child Moving_Jaw, origin xyz=-0.0202 -0.0244 0 rpy=0 3.14 0, axis 0 0 1, limit lower=-0.2 upper=2.0 effort=35 velocity=10
- added joint Pitch: type revolute, parent Rotation_Pitch, child Upper_Arm, origin xyz=0 0.1025 0.0306 rpy=1.5708 0 0, axis 1 0 0, limit lower=-3.14159 upper=0.2 effort=35 velocity=10
- added joint Rotation: type revolute, parent Base, child Rotation_Pitch, origin xyz=0 -0.0452 0.0165 rpy=1.5708 0 0, axis 0 1 0, limit lower=-2.2 upper=2.2 effort=35 velocity=10
- added joint Wrist_Pitch: type revolute, parent Lower_Arm, child Wrist_Pitch_Roll, origin xyz=0 0.0052 0.1349 rpy=-1.5708 0 0, axis 1 0 0, limit lower=-2.0 upper=1.8 effort=35 velocity=10
- added joint Wrist_Roll: type revolute, parent Wrist_Pitch_Roll, child Fixed_Jaw, origin xyz=0 -0.0601 0 rpy=0 1.5708 0, axis 0 1 0, limit lower=-3.14159 upper=3.14159 effort=35 velocity=10
